File: Analog Temp Controller/Analog_Temp_Ctrl.sch (EAGLE design)
At the start: 118 parts, among them IC1 TL074D, IC3 LMV358MMX, IC4 ADA4522-2, J1 USB_MINI-B_SMT, Q1 TIP41C, T1 2N3904, T2 2N3906, U1 ADR01BRZ, U2 ATMEGA32U4-AU, U3 CJT1117-3.3-SOT223, U4 CJT1117-5.0-SOT223, U6 AD5292BRUZ-20, X1 CRYSTAL-3.2-2.5

Commit message: Rev1.1 of CUR CTRL Complete, Ready for Mfg. Temp Ctrl WIP
Parts:
- removed C13: 18pF, rcl:C-EUC0805
- removed C14, C25, C31: 1uF, rcl:C-EUC0805
- removed C15, C19, C20, C24, C26, C27, C29, C32: 0.1uF, rcl:C-EUC0805
- removed C16: 10uF, rcl:CPOL-EUSMCB
- removed C28, C30, C33: 10uF, rcl:C-EUC0805
- removed J1: USB_MINI-B_SMT, SparkFun-Connectors:USB_MINI-B_SMT
- removed JP4: (no value), pinhead:PINHD-2X3
- removed JP8: (no value), pinhead:PINHD-1X3
- removed JP9: (no value), pinhead:PINHD-1X6
- removed L1: MH2029-300Y, SparkFun-Coils:INDUCTOR-0805-3.3UH
- removed R25: 22R, rcl:R-US_R0805
- removed R33, R36, R37, R42: 10K, rcl:R-US_R0805
- removed R34, R35: CG0603MLC-05E, varistor:VARISTORCN0603
- removed R38: 4.7K, rcl:R-US_R0805
- removed RA: Radd, rcl:R-US_R0805
- removed T3: (no value), zetex:PMOSSOT23
- removed U2: ATMEGA32U4-AU, adafruit:ATMEGA32U4-AU
- removed U6: AD5292BRUZ-20, Analog Devices_By_element14_Batch_1:AD5292BRUZ-20
- removed X1: CRYSTAL-3.2-2.5, Arduino_Leonardo-REV3b:CRYSTAL-3.2-2.5
- added C38, C51, C52, C54, C55, C56: 100nF, rcl:C-EUC0805
- added C53: 1uF, rcl:C-EUC0805
- added IC10: 74LVC1G125DCKR, Arduino-M0-V1:INTEGRATEDCIRCUITS_0040_SN74LVC1G125DCKR
- added JP12: (no value), pinhead:PINHD-2X4
- added JP13: (no value), pinhead:PINHD-1X2
- added JP14: (no value), pinhead:PINHD-1X3
- added L4: MH2029-300Y, Arduino-M0-V1:PROTEZIONE_0001_BLM21PG300SN1D_/_MH2029-300Y
- added R56, R63: 330R, rcl:R-US_R0805
- added R57, R58, R59: 10K, rcl:R-US_R0805
- added R60, R61, R62: 100K, rcl:R-US_R0805
- added TR1: PMV48XP, Arduino-M0-V1:TRANSISTORS_0297_PMV48XP
- added U5: ATSAMD21G-A, SparkFun-IC-Microcontroller:ATSAMD21G-A
- added USB: (no value), adafruit:USBMINIB
- added Y1: 32,768Khz_SMD, Arduino-M0-V1:CRISTALLI_0213_ABS07-32.768KHZ-T
- added Z1, Z2: BRNCG0603MLC-05E, Arduino-M0-V1:PROTEZIONE_0010_BRNCG0603MLC-05E
- C11, C23: value 0.1uF -> 10nF
- C12: value 18pF -> 10uF
- F1: value 6V/0.5A -> MF-MSMF050-2 500mA; device SparkFun-Fuses:PPTC_HALF-AMP -> Arduino-M0-V1:PROTEZIONE_0002_MF-MSMF050-2
- JP6: device pinhead:PINHD-2X4 -> pinhead:PINHD-2X3
- R17: value 22R -> (none)
- R4: value 4.7K -> 10K
- S1: value MOMENTARY-SWITCH-SPST-SMD-5.2MM -> MOM SWITCH
Connections:
- removed net DPSS: U2.PE6(INT.6/AIN0), U6.~SYNC
- removed net MISO: JP4.1, U2.PB3(PDO/MISO)
- removed net MOSI: JP4.4, U2.PB2(PDI/MOSI), U6.DIN
- removed net N$2: JP8.3, U2.PF5(ADC5/TMS)
- removed net N$30: JP8.2, U2.PF4(ADC4/TCK)
- removed net N$32: R25.2, U2.D+
- removed net N$33: J1.D-, R17.1, R34.1
- removed net N$36: C11.1, U2.AREF
- removed net N$37: J1.D+, R25.1, R35.1
- removed net N$38: C19.1, IC3A.+IN, R36.1, R37.2
- removed net N$39: JP8.1, U2.PF1(ADC1)
- removed net N$40: R42.2, U2.PE2(!HWB)
- removed net N$41: F1.1, J1.VBUS
- removed net N$43: C12.1, U2.XTAL1, X1.C2
- removed net N$44: C13.1, U2.XTAL2, X1.C1
- removed net N$45: IC3A.OUT, T3.G
- removed net N$47: IC4B.IN+, JP7.1, RA.1
- removed net N$50: C31.2, U6.EXT_CAP
- removed net N$51: C25.2, L1.2, U2.AVCC, U2.AVCC1
- removed net N$53: JP9.6, U2.PD7(OC4D/ADC10/T0)
- removed net N$54: JP9.1, U2.PC6(OC3A/!OC4A)
- removed net N$55: JP9.2, U2.PB7(OC0A/OC1C/RTS)
- removed net N$56: JP9.3, U2.PB6(OC1B/OC4B/ADC13)
- removed net N$57: JP9.4, U2.PB5(OC1A/ADC12/!OC4B)
- removed net N$58: JP9.5, U2.PB4(ADC11)
- removed net N$7: R17.2, U2.D-
- removed net RA: R1.2, R31.1, R32.2, U6.A
- removed net SCK: JP4.3, U2.PB1(SCK), U6.SCLK
- removed net VUSB: C15.2, C16.+, F1.2, T3.D, U2.VBUS
- new net +12V: R60.2
- new net +3V3: C38.1, C51.1, C52.1, IC10P.VDD, JP12.1, JP12.2, L4.2, R4.2, R57.2, R58.2, R62.2, U5.VDDIN, U5.VDDIO@17, U5.VDDIO@36
- new net CS_DAC: U5.PA15(XOUT/SER2:3+)
- new net DCURMON: U5.PB09(AIN3/SER4:1/TC4:1)
- new net DGND: C11.2, C12.1, C23.2, C38.2, C51.2, C52.2, C53.2, C54.2, C55.1, C56.1, IC10P.VSS, JP12.3, JP12.4, JP6.6, R59.1, R61.1, S1.1, U5.GND@18, U5.GND@35, U5.GND@42, U5.GNDANA, USB.GND, Z1.2, Z2.2
- new net ENCA: U5.PA09(I2C/AIN17/SER0:1+)
- new net ENCB: U5.PA08(I2C/AIN16/SER0:0+)
- new net ENCBTN: U5.PA10(AIN18/SER0:2+)
- new net MOSI_DAC: U5.PA13(I2C/SER2:1+)
- new net N$18: C54.1, L4.1, U5.VDDANA
- new net N$52: C55.2, U5.PA00(XIN32/SER1:0/TC2:0), Y1.2
- new net N$59: C56.2, U5.PA01(XOUT32/SER1:1/TC2:1), Y1.1
- new net N$60: U5.PB08(AIN2/SER4:0/TC4:0)
- new net N$61: JP14.3, U5.PA21(SER5:3+)
- new net N$62: JP14.2, U5.PA20(SER5:2+)
- new net N$63: JP14.1, U5.PA19(SER1:3+)
- new net PA02_AIN0: U5.PA02(AIN0/DAC)
- new net PA04_AIN4: JP13.2, U5.PA04(AIN4/REFB/SER0:0/TC0:0)
- new net PA05_AIN5: JP13.1, U5.PA05(AIN5/SER0:1/TC0:1)
- new net PA28_USB_HOST_EN: R63.1, U5.PA28
- new net PB10_S4_SPI_MOSI: JP6.4, U5.PB10(SER4:2+)
- new net PB11_S4_SPI_SCK: JP6.3, U5.PB11(SER4:3+)
- new net PB12_S4_SPI_MISO: JP6.1, U5.PA12(I2C/SER2:0+)
- new net RESET: JP6.5, R4.1, R56.1, S1.2
- new net SCK_DAC: U5.PA14(XIN/SER2:2+)
- new net TARGET_RESET: C23.1, R56.2, U5.!RESET!
- new net TARGET_USB_N: U5.PA24(SER3:2+), USB.D-, Z1.1
- new net TARGET_USB_P: U5.PA25(SER3:3+), USB.D+, Z2.1
- new net USBVCC: C12.2, F1.2, R59.2, TR1.D
- new net USB_ID: IC10A.I, IC10A.OE, R62.1, R63.2, USB.ID
- new net VDDCORE: C53.1, U5.VDDCORE
- new net VIN: U5.PB02(AIN10/SER5:0)
- new net VREG: R1.2, R17.1, R31.1, R32.2
- new net XUSB: C11.1, F1.1, USB.VBUS
- net +15V: no longer C27.1, C28.1, R36.2, U6.VDD
- net +5V: now also JP6.2, TR1.S; no longer C20.1, C23.2, C24.2, C26.2, C32.2, C33.2, IC3P.V+, JP4.2, L1.1, R33.2, T3.S, U2.UVCC, U2.VCC, U2.VCC1, U6.VLOGIC, U6.~RESET
- net -15V: no longer C29.2, C30.2, U6.VSS
- net 3V3: no longer IC3A.-IN, JP6.1, JP6.2, R38.2, R4.2
- net GND: no longer C11.2, C12.2, C13.2, C14.1, C15.1, C16.-, C19.2, C20.2, C23.1, C24.1, C25.1, C26.1, C27.2, C28.2, C29.1, C30.1, C31.1, C32.1, C33.1, IC3P.V-, J1.GND, J1.SHIELD, JP4.6, JP6.3, JP6.4, R34.2, R35.2, R37.1, R42.1, S1.1, U2.GND, U2.GND1, U2.GND2, U2.GND3, U2.UGND, U6.GND, X1.GND@1, X1.GND@2
- net N$46: now also IC10A.O, R60.1, R61.2, TR1.G; no longer C14.2, U2.UCAP
- net RST: no longer JP4.5, R33.1, S1.2, U2./RESET
- net RW: now also IC4B.IN+, JP7.1, R17.2; no longer RA.2, U6.W
- net RXD: no longer U2.PD2(INT2/RXD1)
- net RXLED: no longer U2.PB0(SS)
- net SCL: now also JP12.7, JP12.8, R58.1, U5.PA23(I2C/SER3:0+); no longer JP6.7, JP6.8, R38.1, U2.PD0(INT0/OC0B/SCL)
- net SDA: now also JP12.5, JP12.6, R57.1, U5.PA22(I2C/SER3:0+); no longer JP6.5, JP6.6, R4.1, U2.PD1(INT1/SDA)
- net TXD: no longer U2.PD3(INT3/TXD1)
- net TXLED: no longer U2.PD5(XCK/CTS)
- net UGBOUT: no longer U2.PF0(ADC0)
Other:
- note removed: "DPSS"
- note removed: "Either use 20K Pot(10K NTC) and short Radd or use 100K Pot(100K NTC) and use Radd=50K"
- note removed: "MISO"
- note removed: "MOSI"
- note removed: "N/C"
- note removed: "RA"
- note removed: "RW"
- note removed: "SCK"
- note removed: "SCL"
- note removed: "SDA"
- note removed: "VUSB"

Commit message: Added a Controller for the Pfeiffer IKR/PKR Series Compact Gauges. Temp Ctrl WIP...
Parts:
- removed C17, C18: 10uF, rcl:CPOL-EUSMCB
- removed C21, C22: 1uF, rcl:C-EUC0805
- removed D4: (no value), diode:DIODE-SMB
- removed R39, R40: 1K, rcl:R-US_R0805
- removed RX, TX: (no value), led:LEDCHIPLED_0805
- removed U4: CJT1117-5.0-SOT223, Seeed-IC:PMIC-CJT1117-5.0(SOT223)
- added C13, C14, C33: 10uF, rcl:C-EUC0805
- added C15, C16: 0.1uF, rcl:C-EUC0805
- added IC2: AD620R, analog-devices:AD620R
- added JP4: (no value), pinhead:PINHD-1X2
- added U2: LM1117IMP-3.3, NSC_By_element14_Batch_1.1:LM1117IMP-3.3
- added U6: LM1117IMP-5.0, NSC_By_element14_Batch_1.1:LM1117IMP-5.0
- U3: value CJT1117-3.3-SOT223 -> AD5541; device Seeed-IC:PMIC-CJT1117-3.3(SOT223) -> misc-ics:AD5541
Connections:
- removed net +12V: R60.2
- removed net CS_DAC: U5.PA15(XOUT/SER2:3+)
- removed net MOSI_DAC: U5.PA13(I2C/SER2:1+)
- removed net N$42: R39.1, RX.A
- removed net N$48: R40.1, TX.A
- removed net RXLED: RX.C
- removed net SCK_DAC: U5.PA14(XIN/SER2:2+)
- removed net TXLED: TX.C
- new net DCLK: U3.CLK, U5.PA14(XIN/SER2:2+)
- new net DCS: U3.CS, U5.PA15(XOUT/SER2:3+)
- new net DDATA: U3.DATA, U5.PA13(I2C/SER2:1+)
- new net N$2: JP4.1, R11.2
- new net N$36: IC2.-, U3.VOUT
- new net N$7: C3.1, IC2.+, IC4B.OUT, R6.2
- net +15V: now also C15.2, C33.1, IC2.+V, R60.2, U6.VIN; no longer C18.+, D4.C, U4.IN
- net +3V3: now also C14.1, U2.VOUT, U2.VOUT_2
- net +5V: now also C13.1, U2.VIN, U6.VOUT, U6.VOUT_2; no longer C17.+, C21.1, R39.2, R40.2, U3.IN, U4.OUT
- net -15V: now also C16.1, IC2.-V
- net 3V3: no longer C22.1, U3.OUT
- net DGND: now also C13.2, C14.2, C33.2, PWR.C, U2.ADJ/GND, U3.DGND, U6.ADJ/GND
- net GND: now also C15.1, C16.2, IC2.REF, U3.AGND; no longer C17.-, C18.-, C21.2, C22.2, D4.A, PWR.C, U3.GND, U4.GND
- net N$10: no longer C3.1, IC4B.OUT, R6.2, R8.1
- net N$20: now also JP4.2; no longer R11.2
- net VREG: now also U3.REF, U3.VDD
Other:
- note added: "I ENBL"
- note removed: "RXLED"
- note removed: "TXLED"
- moved on the sheet: C1, C10, C11, C12, C2, C23, C3, C34, C35, C36, C37, C38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

Commit message: Added Pfeiffer G.auge Controller Schematics + FW
Parts:
- removed Z1, Z2: BRNCG0603MLC-05E, Arduino-M0-V1:PROTEZIONE_0010_BRNCG0603MLC-05E
- added H1, H2, H3, H4: MOUNT-PAD-ROUND2.8, holes:MOUNT-PAD-ROUND2.8
- added JP8: JUMPER-SMT_2_NO_SILK, SparkFun-Jumpers:JUMPER-SMT_2_NO_SILK
Connections:
- net DGND: no longer Z1.2, Z2.2
- net GND: now also H1.MOUNT, H2.MOUNT, H3.MOUNT, H4.MOUNT
- net TARGET_USB_N: no longer Z1.1
- net TARGET_USB_P: no longer Z2.1
Changed lines of the file:
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@@
 <part name="C11" library="rcl" library_urn="urn:adsk.eagle:library:334" deviceset="C-EU" device="C0805" package3d_urn="urn:adsk.eagle:package:23617/2" value="10nF"/>
 <part name="SUPPLY3" library="supply2" library_urn="urn:adsk.eagle:library:372" deviceset="DGND" device=""/>
-<part name="Z1" library="Arduino-M0-V1" deviceset="PROTEZIONE_0010_BRNCG0603MLC-05E" device="" value="BRNCG0603MLC-05E"/>
-<part name="Z2" library="Arduino-M0-V1" deviceset="PROTEZIONE_0010_BRNCG0603MLC-05E" device="" value="BRNCG0603MLC-05E"/>
 <part name="SUPPLY4" library="supply2" library_urn="urn:adsk.eagle:library:372" deviceset="DGND" device=""/>
 <part name="C12" library="rcl" library_urn="urn:adsk.eagle:library:334" deviceset="C-EU" device="C0805" package3d_urn="urn:adsk.eagle:package:23617/2" value="10uF"/>
@@
 <part name="P-7" library="supply1" library_urn="urn:adsk.eagle:library:371" deviceset="-15V" device=""/>
 <part name="GND22" library="supply1" library_urn="urn:adsk.eagle:library:371" deviceset="GND" device=""/>
+<part name="H2" library="holes" library_urn="urn:adsk.eagle:library:237" deviceset="MOUNT-PAD-ROUND" device="2.8" package3d_urn="urn:adsk.eagle:package:14281/1"/>
+<part name="H1" library="holes" library_urn="urn:adsk.eagle:library:237" deviceset="MOUNT-PAD-ROUND" device="2.8" package3d_urn="urn:adsk.eagle:package:14281/1"/>
+<part name="H3" library="holes" library_urn="urn:adsk.eagle:library:237" deviceset="MOUNT-PAD-ROUND" device="2.8" package3d_urn="urn:adsk.eagle:package:14281/1"/>
+<part name="H4" library="holes" library_urn="urn:adsk.eagle:library:237" deviceset="MOUNT-PAD-ROUND" device="2.8" package3d_urn="urn:adsk.eagle:package:14281/1"/>
+<part name="GND23" library="supply1" library_urn="urn:adsk.eagle:library:371" deviceset="GND" device=""/>
+<part name="JP8" library="SparkFun-Jumpers" library_urn="urn:adsk.eagle:library:528" deviceset="JUMPER-SMT_2_NO" device="_SILK" package3d_urn="urn:adsk.eagle:package:39279/1"/>
 </parts>
 <sheets>
@@
 <instance part="C11" gate="G$1" x="50.8" y="60.96" rot="R90"/>
 <instance part="SUPPLY3" gate="G$1" x="58.42" y="58.42"/>
-<instance part="Z1" gate="G$1" x="45.72" y="30.48" rot="R90"/>
-<instance part="Z2" gate="G$1" x="58.42" y="30.48" rot="R90"/>
-<instance part="SUPPLY4" gate="G$1" x="58.42" y="17.78"/>
+<instance part="SUPPLY4" gate="G$1" x="40.64" y="17.78"/>
 <instance part="C12" gate="G$1" x="78.74" y="43.18" rot="R180"/>
 <instance part="R59" gate="G$1" x="83.82" y="43.18" rot="R90"/>
@@
 <instance part="SUPPLY1" gate="G$1" x="281.94" y="25.4"/>
 <instance part="P+8" gate="1" x="91.44" y="43.18"/>
+<instance part="H2" gate="G$1" x="302.26" y="203.2"/>
+<instance part="H1" gate="G$1" x="302.26" y="195.58"/>
+<instance part="H3" gate="G$1" x="302.26" y="210.82"/>
+<instance part="H4" gate="G$1" x="302.26" y="218.44"/>
+<instance part="GND23" gate="1" x="297.18" y="185.42"/>
+<instance part="JP8" gate="G$1" x="58.42" y="187.96"/>
 </instances>
 <busses>
@@
 <pinref part="GND44" gate="1" pin="GND"/>
 <wire x1="353.06" y1="139.7" x2="345.44" y2="139.7" width="0.1524" layer="91"/>
+</segment>
+<segment>
+<pinref part="H4" gate="G$1" pin="MOUNT"/>
+<wire x1="299.72" y1="218.44" x2="297.18" y2="218.44" width="0.1524" layer="91"/>
+<wire x1="297.18" y1="218.44" x2="297.18" y2="210.82" width="0.1524" layer="91"/>
+<pinref part="H3" gate="G$1" pin="MOUNT"/>
+<wire x1="297.18" y1="210.82" x2="299.72" y2="210.82" width="0.1524" layer="91"/>
+<wire x1="297.18" y1="210.82" x2="297.18" y2="203.2" width="0.1524" layer="91"/>
+<junction x="297.18" y="210.82"/>
+<pinref part="H2" gate="G$1" pin="MOUNT"/>
+<wire x1="297.18" y1="203.2" x2="299.72" y2="203.2" width="0.1524" layer="91"/>
+<wire x1="297.18" y1="203.2" x2="297.18" y2="195.58" width="0.1524" layer="91"/>
+<junction x="297.18" y="203.2"/>
+<pinref part="H1" gate="G$1" pin="MOUNT"/>
+<wire x1="297.18" y1="195.58" x2="299.72" y2="195.58" width="0.1524" layer="91"/>
+<wire x1="297.18" y1="195.58" x2="297.18" y2="187.96" width="0.1524" layer="91"/>
+<junction x="297.18" y="195.58"/>
+<pinref part="GND23" gate="1" pin="GND"/>
 </segment>
 </net>
@@
 <pinref part="USB" gate="G$1" pin="GND"/>
 <wire x1="30.48" y1="35.56" x2="40.64" y2="35.56" width="0.1524" layer="91"/>
-<wire x1="40.64" y1="35.56" x2="40.64" y2="22.86" width="0.1524" layer="91"/>
-<wire x1="40.64" y1="22.86" x2="45.72" y2="22.86" width="0.1524" layer="91"/>
-<pinref part="Z1" gate="G$1" pin="2"/>
-<wire x1="45.72" y1="22.86" x2="45.72" y2="25.4" width="0.1524" layer="91"/>
-<pinref part="Z2" gate="G$1" pin="2"/>
-<wire x1="45.72" y1="22.86" x2="58.42" y2="22.86" width="0.1524" layer="91"/>
-<wire x1="58.42" y1="22.86" x2="58.42" y2="25.4" width="0.1524" layer="91"/>
-<junction x="45.72" y="22.86"/>
+<wire x1="40.64" y1="35.56" x2="40.64" y2="20.32" width="0.1524" layer="91"/>
 <pinref part="SUPPLY4" gate="G$1" pin="DGND"/>
-<wire x1="58.42" y1="22.86" x2="58.42" y2="20.32" width="0.1524" layer="91"/>
-<junction x="58.42" y="22.86"/>
 </segment>
 <segment>
@@
 <wire x1="30.48" y1="43.18" x2="58.42" y2="43.18" width="0.1524" layer="91"/>
 <label x="40.64" y="43.18" size="1.778" layer="95"/>
-<pinref part="Z2" gate="G$1" pin="1"/>
-<wire x1="58.42" y1="35.56" x2="58.42" y2="43.18" width="0.1524" layer="91"/>
 </segment>
 </net>
@@
 <segment>
 <pinref part="USB" gate="G$1" pin="D-"/>
-<wire x1="30.48" y1="40.64" x2="45.72" y2="40.64" width="0.1524" layer="91"/>
+<wire x1="30.48" y1="40.64" x2="58.42" y2="40.64" width="0.1524" layer="91"/>
 <label x="40.64" y="40.64" size="1.778" layer="95"/>
-<pinref part="Z1" gate="G$1" pin="1"/>
-<wire x1="45.72" y1="40.64" x2="58.42" y2="40.64" width="0.1524" layer="91"/>
-<wire x1="45.72" y1="35.56" x2="45.72" y2="40.64" width="0.1524" layer="91"/>
-<junction x="45.72" y="40.64"/>
-</segment>
-</net>
+</segment>
+</net>
