File: Pfeiffer_Compact_Gauge_Controller/Pfeiffer_Compact_Gauge_Controller.sch (EAGLE design)
At the start: 53 parts, among them IC1 TL072D, U1 ATMEGA32U4-AU, U6 LM1117IMP-5.0

Commit message: Added Pfeiffer G.auge Controller Schematics + FW
Parts:
- removed TR1, TR2: PMV48XP, Arduino-M0-V1:TRANSISTORS_0297_PMV48XP
- added D1: 1A/40V/500mV, SparkFun-DiscreteSemi:DIODE-SCHOTTKY-SS14
- added JP7: (no value), pinhead:PINHD-1X2
- added R14: OPEN, rcl:R-US_R0805
- R7: value 10K -> 11K
- R9: value 10K -> 0R
- U6: value LM1117IMP-5.0 -> LM340A
Connections:
- net +24V: now also C16.1, U6.VIN; no longer TR1.G, TR2.D
- net +5V: now also D1.C; no longer TR1.S, TR2.G
- net GND: now also R14.1, R8.2; no longer R8.1
- net N$10: now also R7.2, R8.1; no longer R7.1
- net N$12: now also D1.A, JP7.1; no longer C16.1, TR2.S, U6.VIN
- net N$9: now also R14.2; no longer R8.2
- net SIGNAL: now also R7.1; no longer R7.2
- net VUSB: now also JP7.2; no longer TR1.D
Other:
- moved on the sheet: R7, R8
