File: Pfeiffer_Compact_Gauge_Controller/Pfeiffer_Compact_Gauge_Controller.brd (EAGLE design)
At the start: 52 x 59 mm, 53 parts, among them IC1 TL072D, U1 ATMEGA32U4-AU, U6 LM1117IMP-5.0

Commit message: Added Pfeiffer G.auge Controller Schematics + FW
Parts:
- removed TR1, TR2: PMV48XP, Arduino-M0-V1:TRANSISTORS_SOT-23
- added D1: 1A/40V/500mV, SparkFun-DiscreteSemi:SMA-DIODE
- added JP7: (no value), pinhead:1X02
- added R14: OPEN, rcl:R0805
- R7: value 10K -> 11K
- R9: value 10K -> 0R
- U6: value LM1117IMP-5.0 -> LM340A
- moved C15 14.0 mm to (29.8, 47.9), turned to 90 degrees
- moved R59 10.9 mm to (32.1, 47.9), turned to 90 degrees
- moved R8 2.37 mm to (27.7, 11.6), turned to 180 degrees
- moved F1 1.76 mm to (36.7, 47.8), turned to 180 degrees
- moved U6 1.65 mm to (28.4, 41.5)
- moved R7 1.09 mm to (27.7, 13.8), turned to 0 degrees
- moved C9 0.90 mm to (23.0, 35.4), turned to 0 degrees
- moved JP2 0.64 mm to (22.9, 14.0)
- moved 5V 0.63 mm to (23.0, 38.1)
- moved C17 0.57 mm to (27.4, 35.4)
- moved C14 0.40 mm to (41.1, 47.5)
- moved C12 0.38 mm to (32.8, 36.6)
- moved C16 0.25 mm to (35.1, 36.6)
- moved R10 0.13 mm to (37.3, 36.6)
Connections:
- net +24V: now also C16.1, U6.3; no longer TR1.3, TR2.1
- net +5V: now also D1.C; no longer TR1.2, TR2.3
- net GND: now also R14.1, R8.2; no longer R8.1
- net N$10: now also R7.2, R8.1; no longer R7.1
- net N$12: now also D1.A, JP7.1; no longer C16.1, TR2.2, U6.3
- net N$9: now also R14.2; no longer R8.2
- net SIGNAL: now also R7.1; no longer R7.2
- net VUSB: now also JP7.2; no longer TR1.1
Routing:
- net VUSB: track 48.0 -> 43.8 mm
- net +24V: track 73.1 -> 69.7 mm
- net N$10: track 2.86 -> 5.32 mm
- net N$12: track 5.84 -> 3.77 mm
- net XUSB: track 7.65 -> 6.33 mm
- net SIGNAL: track 30.4 -> 31.1 mm
- net N$13: track 15.8 -> 16.5 mm
- net N$9: track 6.18 -> 6.82 mm
- net N$11: track 15.8 -> 16.5 mm
- net N$16: track 2.29 -> 2.93 mm
Other:
- board text added: "J1"
